File: hardware/controller.sch (EAGLE design)
At the start: 27 parts, among them IC3 TS5205, J1 PIN2F061.100, J2 PIN2F061.100, J3 PIN2F061.100, K1 G5LE, K2 G5LE, Q1 ABM8G, Q2 BC846ASMD, Q3 BC846ASMD, X1 FCI-USB-MICRO-B

Commit message: hardware: first attempt with triacs
Parts:
- removed D3: BAT54C, diode:BAT54C
- removed K1, K2: G5LE, relay:G5LE
- removed Q3: BC846ASMD, transistor-npn:BC846ASMD
- added B1: MB6S, rectifier:MB6S
- added C7, C8: 1nF, resistor:C-USC0402K
- added D1: (no value), diode:DIODE-SOD80C
- added J4: PIN2F061.100, con-faston:PIN2F061.100
- added OK1: 4N35SM, optocoupler:4N35SM
- added R10: 44kΩ, resistor:R-US_R0402
- added R11: 1kΩ, resistor:R-US_R0402
- added R4, R5, R6, R7: 33Ω, resistor:R-US_R0402
- added R8, R9: 440kΩ, resistor:R-US_R0402
- added U$4, U$5: MOC3063, crawford:MOC3063
- added U$6, U$7: BT137S-600D, crawford:BT137S-600D
- Q2: value BC846ASMD -> BC817-40SMD; device transistor-npn:BC846ASMD -> transistor-npn:BC817-40SMD
Connections:
- removed net B_K1: Q3.B, U$1.P0.7/!CTS!
- removed net B_K2: Q2.B, U$1.P1.28/CT32B0_CAP0/SCLK
- new net INT_ZX: OK1.COL, U$1.P0.4/SCL
- new net N$12: J1.1, R6.2, U$6.A2
- new net N$13: U$4.A1, U$6.G
- new net N$14: U$5.A1, U$7.G
- new net N$15: B1.-, C8.1, R10.1, R11.1
- new net N$16: B1.+, D1.C, Q2.B, R10.2
- new net N$17: B1.AC1, C7.1, R9.2
- new net N$18: B1.AC2, C7.2, R8.2
- new net N$19: OK1.A, R11.2
- new net N$20: OK1.C, Q2.C
- new net N$21: C8.2, D1.A, Q2.E
- new net N$23: U$4.C
- new net N$24: U$5.C
- new net V+: J3.1, R8.1
- new net V-: J4.1, R9.1, U$6.A1, U$7.A1
- net +3V3: now also R4.1, R5.1; no longer D3.CC, K11.1, K21.1
- net CS: no longer U$1.P1.21/!DCD!/MISO1
- net GND: now also OK1.EMI; no longer Q2.E, Q3.E
- net N$1: now also R6.1, U$4.A2; no longer J2.1, K12.P, K22.P
- net N$10: now also R4.2, U$4.A; no longer D3.A2, K11.2, Q3.C
- net N$11: now also R5.2, U$5.A; no longer D3.A1, K21.2, Q2.C
- net N$2: now also J2.1, R7.2, U$7.A2; no longer J3.1, K22.S
- net N$8: now also R7.1, U$5.A2; no longer J1.1, K12.S
- net SCK: no longer U$1.P0.8/MISO0/CT16B0_MAT0
- net SO: no longer U$1.P1.31
Other:
- moved on the sheet: J1, J2, J3, Q2, U$2, U$3
